File: hardware/bsidesorl-v1.kicad_sch (KiCad schematic)
At the start: 35 parts, among them J1 SAO Connector, Q1 SI2302S, SW1 MST22D18G2_125, U1 CH32V003F4P6, U2 TPS61021ADSGR

Commit message: Production PCB as ordered
* Fingerprint soldermask artwork and board outline sources
* SW1 excluded from BOM/CPL (hand-placed)
* Regenerated JLCPCB gerbers and production files
* Add mk_easyeda.py for importing the KiCad board into EasyEDA Pro
* Ignore local fab/order artifacts

Co-Authored-By: Claude Opus 5.5 (1M context) <noreply@anthropic.com>
Claude-Session: https://claude.ai/code/session_01VwuCpwoY4XUvmQLYcHynUX
Parts:
- SW1: now left out of the parts list
Changed lines of the file:
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@@
 		(body_style 1)
 		(exclude_from_sim no)
-		(in_bom yes)
+		(in_bom no)
 		(on_board yes)
-		(in_pos_files yes)
+		(in_pos_files no)
 		(dnp no)
 		(property "Reference" "SW1"
